File: rele cc y bg/rele cc y bg.kicad_pcb (KiCad board)
At the start: 2 copper layers, 41 parts, among them J1 Screw_Terminal_01x03, J2 Screw_Terminal_01x03, J3 Screw_Terminal_01x03, J4 Conn_01x06_Pin, J5 Screw_Terminal_01x03, J6 Screw_Terminal_01x02, K1 RELAY_C, K2 RELAY_C, K3 RELAY_C, K5 RELAY_C, Q1 2N2222, Q2 2N2222, Q3 2N2222, Q4 2N2222, U1 EL817, U2 EL817, U4 EL817, U5 EL817, U6 L7805, U8 ESP32_DEVKITC

Commit message: V3
Parts:
- J1, J2, J3, J5: footprint Connector_Wuerth:Wuerth_WR-WTB_64800311622_1x03_P1.50mm_Vertical -> EESTN5:BORNERA3_AZUL
- moved Q4 181.9 mm to (34.8, 45.9)
- moved Q1 172.9 mm to (35.1, 69.5)
- moved Q3 171.9 mm to (35.3, 117.8)
- moved Q2 171.3 mm to (35.1, 94.5)
- moved D6 162.0 mm to (23.6, 50.0), turned to -90 degrees
- moved D2 151.3 mm to (24.1, 73.9), turned to -90 degrees
- moved K5 150.8 mm to (49.6, 49.6), turned to 90 degrees
- moved J5 148.1 mm to (63.5, 122.4), turned to -90 degrees
- moved D3 148.0 mm to (23.4, 98.7), turned to -90 degrees
- moved D8 146.3 mm to (24.1, 123.0), turned to -90 degrees
- moved D4 144.9 mm to (30.4, 39.3), turned to 180 degrees
- moved J3 140.9 mm to (64.4, 72.0), turned to -90 degrees
- moved J1 140.8 mm to (65.1, 49.7), turned to -90 degrees
- moved R5 139.9 mm to (26.9, 39.4), turned to 180 degrees
- moved D5 139.8 mm to (38.2, 39.3), turned to 180 degrees
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Connections:
- C2 pad 1: Net-(U6-OUT) -> +5V
- D2 pad 1: Net-(D2-K) -> +5V
- D3 pad 1: Net-(D2-K) -> +5V
- D6 pad 1: Net-(D6-K) -> +5V
- D8 pad 1: Net-(D2-K) -> +5V
- K1 pad 5: Net-(D2-K) -> +5V
- K2 pad 5: Net-(D2-K) -> +5V
- K3 pad 5: Net-(D2-K) -> +5V
- K5 pad 5: Net-(D6-K) -> +5V
- R5 pad 2: Net-(D6-K) -> +5V
- R6 pad 2: Net-(D6-K) -> +5V
- R8 pad 2: VCC -> IN3
- U1 pad 4: Net-(D2-K) -> +5V
- U2 pad 4: Net-(D2-K) -> +5V
- U4 pad 4: Net-(D2-K) -> +5V
- U5 pad 4: Net-(D6-K) -> +5V
- U6 pad 3: Net-(U6-OUT) -> +5V
- U8 pad 1: Net-(U6-OUT) -> unconnected-(U8-3V3-Pad1)
- U8 pad 19: unconnected-(U8-5V-Pad19) -> +5V
- U8 pad 5: IN1 -> IN4
- U8 pad 6: IN2 -> IN3
- U8 pad 7: IN3 -> IN2
- U8 pad 8: IN4 -> IN1
Routing:
- net +5V: track 0.00 -> 180.7 mm
- net IN3: track 0.00 -> 126.2 mm
- net IN1: track 0.00 -> 96.9 mm
- net IN2: track 0.00 -> 92.5 mm
- net Net-(D5-K): track 0.00 -> 38.0 mm
- net Net-(J3-Pin_3): track 0.00 -> 32.5 mm
- net Net-(J1-Pin_3): track 0.00 -> 31.7 mm
- net Net-(J2-Pin_3): track 0.00 -> 31.5 mm
- net Net-(D2-A): track 0.00 -> 31.0 mm
- net Net-(J5-Pin_3): track 0.00 -> 30.5 mm
- net Net-(J6-Pin_1): track 0.00 -> 28.8 mm
- net Net-(D3-A): track 0.00 -> 27.5 mm
- net Net-(D2-K): track 26.3 -> 0.00 mm
- net Net-(D8-A): track 0.00 -> 25.6 mm
- net Net-(J3-Pin_1): track 0.00 -> 20.4 mm
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